Commit message: Finished Quadruped

File: generated/body.urdf (robot description, URDF)
Before this commit: robot robot, 3 links, 2 joints
Links:
- added link BackLower, mass 1; collision box size=0.2 0.2 1; visual box size=0.2 0.2 1
- added link FrontLower, mass 1; collision box size=0.2 0.2 1; visual box size=0.2 0.2 1
- added link LeftLeg, mass 1; collision box size=1 0.2 0.2; visual box size=1 0.2 0.2
- added link LeftLower, mass 1; collision box size=0.2 0.2 1; visual box size=0.2 0.2 1
- added link RightLeg, mass 1; collision box size=1 0.2 0.2; visual box size=1 0.2 0.2
- added link RightLower, mass 1; collision box size=0.2 0.2 1; visual box size=0.2 0.2 1
- link BackLeg: geometry collision box size=0.2 1 0.2; visual box size=0.2 1 0.2
- link FrontLeg: geometry collision box size=0.2 1 0.2; visual box size=0.2 1 0.2
Joints:
- added joint BackLeg_BackLower: type revolute, parent BackLeg, child BackLower, origin xyz=0 -1 0 rpy=0 0 0, axis 1 0 0, limit lower=-3.14159 upper=3.14159 effort=0.0 velocity=0.0
- added joint FrontLeg_FrontLower: type revolute, parent FrontLeg, child FrontLower, origin xyz=0 1 0 rpy=0 0 0, axis 1 0 0, limit lower=-3.14159 upper=3.14159 effort=0.0 velocity=0.0
- added joint LeftLeg_LeftLower: type revolute, parent LeftLeg, child LeftLower, origin xyz=-1 0 0 rpy=0 0 0, axis 0 1 0, limit lower=-3.14159 upper=3.14159 effort=0.0 velocity=0.0
- added joint RightLeg_RightLower: type revolute, parent RightLeg, child RightLower, origin xyz=1 0 0 rpy=0 0 0, axis 0 1 0, limit lower=-3.14159 upper=3.14159 effort=0.0 velocity=0.0
- added joint Torso_LeftLeg: type revolute, parent Torso, child LeftLeg, origin xyz=-0.5 0 1 rpy=0 0 0, axis 0 1 0, limit lower=-3.14159 upper=3.14159 effort=0.0 velocity=0.0
- added joint Torso_RightLeg: type revolute, parent Torso, child RightLeg, origin xyz=0.5 0 1 rpy=0 0 0, axis 0 1 0, limit lower=-3.14159 upper=3.14159 effort=0.0 velocity=0.0
- joint Torso_BackLeg: axis 0 1 0 -> 1 0 0; origin xyz=0.5 0 1 rpy=0 0 0 -> xyz=0 -0.5 1 rpy=0 0 0
- joint Torso_FrontLeg: axis 0 1 0 -> 1 0 0; origin xyz=-0.5 0 1 rpy=0 0 0 -> xyz=0 0.5 1 rpy=0 0 0

Commit message: Made new biped

File: generated/body.urdf (robot description, URDF)
Before this commit: robot robot, 9 links, 8 joints
Links:
- removed link BackLeg
- removed link BackLower
- removed link FrontLeg
- removed link FrontLower
- added link LeftFoot, mass 1; collision box size=0.5 0.5 0.1; visual box size=0.5 0.5 0.1
- added link RightFoot, mass 1; collision box size=0.5 0.5 0.1; visual box size=0.5 0.5 0.1
- link LeftLeg: geometry collision box size=0.2 0.2 0.7; visual box size=0.2 0.2 0.7
- link LeftLower: geometry collision box size=0.2 0.2 0.7; visual box size=0.2 0.2 0.7
- link RightLeg: geometry collision box size=0.2 0.2 0.7; visual box size=0.2 0.2 0.7
- link RightLower: geometry collision box size=0.2 0.2 0.7; visual box size=0.2 0.2 0.7
Joints:
- removed joint BackLeg_BackLower
- removed joint FrontLeg_FrontLower
- removed joint Torso_BackLeg
- removed joint Torso_FrontLeg
- added joint LeftLower_LeftFoot: type revolute, parent LeftLower, child LeftFoot, origin xyz=0 0 -0.35 rpy=0 0 0, axis 1 0 0, limit lower=-3.14159 upper=3.14159 effort=0.0 velocity=0.0
- added joint RightLower_RightFoot: type revolute, parent RightLower, child RightFoot, origin xyz=0 0 -0.35 rpy=0 0 0, axis 1 0 0, limit lower=-3.14159 upper=3.14159 effort=0.0 velocity=0.0
- joint LeftLeg_LeftLower: axis 0 1 0 -> 1 0 0; origin xyz=-1 0 0 rpy=0 0 0 -> xyz=0 0 -0.35 rpy=0 0 0
- joint RightLeg_RightLower: axis 0 1 0 -> 1 0 0; origin xyz=1 0 0 rpy=0 0 0 -> xyz=0 0 -0.35 rpy=0 0 0
- joint Torso_LeftLeg: axis 0 1 0 -> 1 0 0; origin xyz=-0.5 0 1 rpy=0 0 0 -> xyz=-0.6 0 1.5 rpy=0 0 0
- joint Torso_RightLeg: axis 0 1 0 -> 1 0 0; origin xyz=0.5 0 1 rpy=0 0 0 -> xyz=0.6 0 1.5 rpy=0 0 0

Commit message: Snake be movin

File: generated/body.urdf (robot description, URDF)
Before this commit: robot robot, 7 links, 6 joints
Links:
- removed link LeftFoot
- removed link LeftLeg
- removed link LeftLower
- removed link RightFoot
- removed link RightLeg
- removed link RightLower
- removed link Torso
- added link link0, mass 1; collision box size=0.5241860896300164 0.3149064069468921 0.5527679749422072; visual box size=0.5241860896300164 0.3149064069468921 0.5527679749422072
- added link link1, mass 1; collision box size=0.876740566811403 0.7744892190915794 0.39892339540008576; visual box size=0.876740566811403 0.7744892190915794 0.39892339540008576
- added link link2, mass 1; collision box size=0.5557399197068735 0.6245772676999037 0.7405974349245488; visual box size=0.5557399197068735 0.6245772676999037 0.7405974349245488
- added link link3, mass 1; collision box size=0.592338986420841 0.7843453401340477 0.33081950618534833; visual box size=0.592338986420841 0.7843453401340477 0.33081950618534833
Joints:
- removed joint LeftLeg_LeftLower
- removed joint LeftLower_LeftFoot
- removed joint RightLeg_RightLower
- removed joint RightLower_RightFoot
- removed joint Torso_LeftLeg
- removed joint Torso_RightLeg
- added joint link0_link1: type revolute, parent link0, child link1, origin xyz=0.2620930448150082 0 0.5 rpy=0 0 0, axis 0 1 0, limit lower=-3.14159 upper=3.14159 effort=0.0 velocity=0.0
- added joint link1_link2: type revolute, parent link1, child link2, origin xyz=0.876740566811403 0 0 rpy=0 0 0, axis 0 1 0, limit lower=-3.14159 upper=3.14159 effort=0.0 velocity=0.0
- added joint link2_link3: type revolute, parent link2, child link3, origin xyz=0.5557399197068735 0 0 rpy=0 0 0, axis 0 1 0, limit lower=-3.14159 upper=3.14159 effort=0.0 velocity=0.0

Commit message: Test

File: generated/body.urdf (robot description, URDF)
Before this commit: robot robot, 4 links, 3 joints
Links:
- added link link4, mass 1; collision box size=0.5432191459748329 0.4069625573933822 0.3535920357644838; visual box size=0.5432191459748329 0.4069625573933822 0.3535920357644838
- link link0: geometry collision box size=0.8998290181969226 0.5129145751138855 0.37231971473513414; visual box size=0.8998290181969226 0.5129145751138855 0.37231971473513414
- link link1: geometry collision box size=0.40746381816264576 0.7857322662150767 0.44422641949325503; visual box size=0.40746381816264576 0.7857322662150767 0.44422641949325503
- link link2: geometry collision box size=0.5238726348481337 0.5704633361873276 0.6108741511404225; visual box size=0.5238726348481337 0.5704633361873276 0.6108741511404225
- link link3: geometry collision box size=0.40231330137865995 0.6597916331256237 0.7082687757849204; visual box size=0.40231330137865995 0.6597916331256237 0.7082687757849204
Joints:
- added joint link3_link4: type revolute, parent link3, child link4, origin xyz=0.40231330137865995 0 0 rpy=0 0 0, axis 0 1 0, limit lower=-3.14159 upper=3.14159 effort=0.0 velocity=0.0
- joint link0_link1: origin xyz=0.2620930448150082 0 0.5 rpy=0 0 0 -> xyz=0.4499145090984613 0 0.5 rpy=0 0 0
- joint link1_link2: origin xyz=0.876740566811403 0 0 rpy=0 0 0 -> xyz=0.40746381816264576 0 0 rpy=0 0 0
- joint link2_link3: origin xyz=0.5557399197068735 0 0 rpy=0 0 0 -> xyz=0.5238726348481337 0 0 rpy=0 0 0

Commit message: Done

File: generated/body.urdf (robot description, URDF)
Before this commit: robot robot, 5 links, 4 joints
Links:
- added link link5, mass 1; collision box size=0.9079560460450131 0.8770441311012365 0.48877438884496943; visual box size=0.9079560460450131 0.8770441311012365 0.48877438884496943
- added link link6, mass 1; collision box size=0.5756144474225906 0.8951389733324557 0.5425354323806582; visual box size=0.5756144474225906 0.8951389733324557 0.5425354323806582
- link link0: geometry collision box size=0.8257277125348907 0.5088962880423924 0.33157533444188014; visual box size=0.8257277125348907 0.5088962880423924 0.33157533444188014
- link link1: geometry collision box size=0.5468438042431271 0.3332147747309436 0.4429507518879952; visual box size=0.5468438042431271 0.3332147747309436 0.4429507518879952
- link link2: geometry collision box size=0.8931703139545673 0.3210502521609692 0.734522228725448; visual box size=0.8931703139545673 0.3210502521609692 0.734522228725448
- link link3: geometry collision box size=0.6951708526784068 0.7265655636519048 0.5191760870539817; visual box size=0.6951708526784068 0.7265655636519048 0.5191760870539817
- link link4: geometry collision box size=0.7778113748473707 0.6622664674579682 0.5526323100697617; visual box size=0.7778113748473707 0.6622664674579682 0.5526323100697617
Joints:
- added joint link4_link5: type revolute, parent link4, child link5, origin xyz=0.7778113748473707 0 0 rpy=0 0 0, axis 0 1 0, limit lower=-3.14159 upper=3.14159 effort=0.0 velocity=0.0
- added joint link5_link6: type revolute, parent link5, child link6, origin xyz=0.9079560460450131 0 0 rpy=0 0 0, axis 0 1 0, limit lower=-3.14159 upper=3.14159 effort=0.0 velocity=0.0
- joint link0_link1: origin xyz=0.4499145090984613 0 0.5 rpy=0 0 0 -> xyz=0.4128638562674454 0 0.5 rpy=0 0 0
- joint link1_link2: origin xyz=0.40746381816264576 0 0 rpy=0 0 0 -> xyz=0.5468438042431271 0 0 rpy=0 0 0
- joint link2_link3: origin xyz=0.5238726348481337 0 0 rpy=0 0 0 -> xyz=0.8931703139545673 0 0 rpy=0 0 0
- joint link3_link4: origin xyz=0.40231330137865995 0 0 rpy=0 0 0 -> xyz=0.6951708526784068 0 0 rpy=0 0 0

Commit message: Made Class Generator for Random Bodies

File: generated/body.urdf (robot description, URDF)
Before this commit: robot robot, 7 links, 6 joints
Links:
- removed link link3
- removed link link4
- removed link link5
- removed link link6
- link link0: geometry collision box size=0.8450099203277692 0.4030195561385245 0.8198738861892394; visual box size=0.8450099203277692 0.4030195561385245 0.8198738861892394
- link link1: geometry collision box size=0.8349059488761257 0.8043280033889657 0.33450467746856416; visual box size=0.8349059488761257 0.8043280033889657 0.33450467746856416
- link link2: geometry collision box size=0.5907469400891178 0.694286694201677 0.6377173949275491; visual box size=0.5907469400891178 0.694286694201677 0.6377173949275491
Joints:
- removed joint link2_link3
- removed joint link3_link4
- removed joint link4_link5
- removed joint link5_link6
- joint link0_link1: origin xyz=0.4128638562674454 0 0.5 rpy=0 0 0 -> xyz=0.4225049601638846 0 0.5 rpy=0 0 0
- joint link1_link2: origin xyz=0.5468438042431271 0 0 rpy=0 0 0 -> xyz=0.8349059488761257 0 0 rpy=0 0 0
