Commit message: Testing

File: generated/body0.urdf (robot description, URDF)
Before this commit: robot robot, 3 links, 2 joints
Links:
- removed link torso2
- link torso0: geometry collision box size=0.54986119643516 0.875590032493996 0.6700706148249028; visual box size=0.54986119643516 0.875590032493996 0.6700706148249028
- link torso1: geometry collision box size=0.9952221256564993 0.7481750608045294 0.6476863938233011; visual box size=0.9952221256564993 0.7481750608045294 0.6476863938233011
Joints:
- removed joint torso0_torso2
- joint torso0_torso1: origin xyz=0.0 0.3053908700557122 1.4973268511309308 rpy=0 0 0 -> xyz=0.27493059821758 -0.437795016246998 0.6700706148249028 rpy=0 0 0

Commit message: Assignment 8

File: generated/body0.urdf (robot description, URDF)
Before this commit: robot robot, 2 links, 1 joints
Links:
- added link torso2, mass 1; collision box size=0.6890562782679608 0.6906331411116989 0.8226853714344253; visual box size=0.6890562782679608 0.6906331411116989 0.8226853714344253
- added link torso3, mass 1; collision box size=0.9735126891339533 0.9509633696399695 0.7454172271367179; visual box size=0.9735126891339533 0.9509633696399695 0.7454172271367179
- link torso0: geometry collision box size=0.9143859813659128 0.8298342326242525 0.7738669953580465; visual box size=0.9143859813659128 0.8298342326242525 0.7738669953580465
- link torso1: geometry collision box size=0.6117532251464759 0.7962660668847045 0.6713300779526274; visual box size=0.6117532251464759 0.7962660668847045 0.6713300779526274
Joints:
- added joint torso0_torso3: type revolute, parent torso0, child torso3, origin xyz=-0.4571929906829564 -0.41491711631212624 0.7454172271367177 rpy=0 0 0, axis 0 1 0, limit lower=-3.14159 upper=3.14159 effort=0.0 velocity=0.0
- added joint torso1_torso2: type revolute, parent torso1, child torso2, origin xyz=0.4571929906829564 -0.41491711631212624 0.38693349767902324 rpy=0 0 0, axis 0 1 0, limit lower=-3.14159 upper=3.14159 effort=0.0 velocity=0.0
- joint torso0_torso1: origin xyz=0.27493059821758 -0.437795016246998 0.6700706148249028 rpy=0 0 0 -> xyz=0.4571929906829564 0.41491711631212624 0.7454172271367177 rpy=0 0 0

Commit message: Initial Commit

File: generated/body0.urdf (robot description, URDF)
Before this commit: robot robot, 2 links, 1 joints
Links:
- link torso0: geometry collision box size=0.7402846252169596 0.7935535112319546 0.9493831380473489; visual box size=0.7402846252169596 0.7935535112319546 0.9493831380473489
- link torso1: geometry collision box size=0.5025654538168687 0.7863778796887982 0.5199824193136828; visual box size=0.5025654538168687 0.7863778796887982 0.5199824193136828
Joints:
- joint torso0_torso1: origin xyz=0.27493059821758 -0.437795016246998 0.6700706148249028 rpy=0 0 0 -> xyz=-0.3701423126084798 -0.3967767556159773 0.9493831380473489 rpy=0 0 0
